File: hardware/board_pcb/medipix.sch (EAGLE design)
At the start: 106 parts, among them IC1 AVR_XMEGA_A4U44A, IC2 FM25H20, U1 IRF7313, U10 BSS138AKA, U11 IRF7313, U12 BSS138AKA, U13 BSS138AKA, U14 BSS84, U15 IRF7319, U16 BSS138AKA, U17 BSS138AKA, U2 IRF7328, U3 IRF7328, U4 BSS84, U5 IRF7313, U6 IRF7328, U7 BSS84, U8 BSS84, U9 BSS138AKA

Commit message: + new connectors, + medipix 2.2V switch
Parts:
- removed GND2: GND, medipix:PIN
- removed MISO: MISO, medipix:PIN
- removed MOSI: MOSI, medipix:PIN
- removed SCK: SCK, medipix:PIN
- removed SCL: SCL, medipix:PIN
- removed SDA: SDA, medipix:PIN
- removed U$1, U$3, U$4, U$5, U$6, UART: MOLEX-MICROBLADE-4, medipix:MOLEX-MICROBLADE-4
- added P1, P2: 53398-0310, con-molex-picoblade:53398-0310
- added P3: 53398-0510, con-molex-picoblade:53398-0510
- added R34, R35: 1k, medipix:RESISTOR0805
- added R36, R37: 100k, medipix:RESISTOR0805
- added TXD1: IN, medipix:PIN
- added TXD2: OUT, medipix:PIN
- added U18: IRF7319, medipix:IRF7319
Connections:
- removed net GND: C1.P$2, C10.P$1, C11.P$1, C12.P$1, C13.P$1, C14.P$1, C15.P$1, C19.P$2, C2.P$2, C20.P$2, C21.P$2, C22.C_EL-, C23.P$1, C24.P$1, C25.P$1, C26.P$2, C27.P$2, C28.C_EL-, C29.C_EL-, C3.P$1, C4.C_EL-, C5.P$1, C6.C_EL-, C8.P$1, C9.P$1, GND.D, GND1.D, GND2.D, H2.H2-34, H2.H2-36, IC1.AGND, IC1.GND1, IC1.GND2, IC1.GND3, IC2.VSS, MP.GND, R10.P$2, R12.P$1, R18.P$2, R21.P$2, R25.P$2, R26.P$2, R5.P$2, R6.P$2, R7.P$1, U$1.GND, U$3.GND, U$4.GND, U$5.GND, U$6.GND, U1.S1, U1.S2, U10.S, U11.S1, U11.S2, U12.S, U13.S, U15.S1, U5.S1, U5.S2, U9.S, UART.GND
- removed net N$14: IC1.PD5, MOSI.D
- removed net N$15: IC1.PD6, MISO.D
- removed net N$16: IC1.PD7, SCK.D
- removed net SCL_C: IC1.PC1, SCL.D, U$6.M1
- removed net SDA_C: IC1.PC0, SDA.D, U$6.M2
- new net GNDD: C1.P$2, C10.P$1, C11.P$1, C12.P$1, C13.P$1, C14.P$1, C15.P$1, C19.P$2, C2.P$2, C20.P$2, C21.P$2, C22.C_EL-, C23.P$1, C24.P$1, C25.P$1, C26.P$2, C27.P$2, C28.C_EL-, C29.C_EL-, C3.P$1, C4.C_EL-, C5.P$1, C6.C_EL-, C8.P$1, C9.P$1, GND.D, GND1.D, H2.H2-34, H2.H2-36, IC1.AGND, IC1.GND1, IC1.GND2, IC1.GND3, IC2.VSS, MP.GND, P1.3, P2.3, P3.1, R10.P$2, R12.P$1, R18.P$2, R21.P$2, R25.P$2, R26.P$2, R36.P$2, R5.P$2, R6.P$2, R7.P$1, U1.S1, U1.S2, U10.S, U11.S1, U11.S2, U12.S, U13.S, U15.S1, U18.S1, U5.S1, U5.S2, U9.S
- new net MEDIPIX-SW2: IC1.PD7, R36.P$1, U18.G1
- new net MEDIPIX_GATE2: R37.P$1, U18.D1, U18.D12, U18.G2
- new net MPX2.2IN: R37.P$2, TXD1.D, U18.S2
- new net MPX2.2OUT: TXD2.D, U18.D2, U18.D22
- new net N$9: MP.TXD, R34.P$2
- new net RXDMMM: MP.RXD, R35.P$2
- net +3.3V: now also P1.1, P2.1, P3.2; no longer U$1.+3V, U$3.+3V, U$4.+3V, U$5.+3V, U$6.+3V, UART.+3V
- net N$10: no longer UART.M2
- net N$11: no longer UART.M1
- net PA0: now also P3.5; no longer U$4.M1
- net PA1: now also P3.4; no longer U$4.M2
- net PA2: now also P3.3; no longer U$3.M1
- net PA3: now also P1.2; no longer U$3.M2
- net PA4: now also P2.2; no longer U$5.M1
- net PA5: no longer U$5.M2
- net PA6: no longer U$1.M1
- net PA7: no longer U$1.M2
- net RXDM: now also R35.P$1; no longer MP.RXD
- net TXDM: now also R34.P$1; no longer MP.TXD

Commit message: + Board updated with temperature sensor connector
Parts:
- removed RXD0: RX, medipix:PIN
- removed TXD0: TX, medipix:PIN
- added GND25: +3.3, medipix:PIN
- added GND28: +5, medipix:PIN
- added U$1: THERM, medipix:THERM
- P1, P2: value 53398-0310 -> PICOBLADE
- P3: value 53398-0510 -> PICOBLADE
Connections:
- removed net N$10: IC1.PD3, TXD0.D
- removed net N$11: IC1.PD2, RXD0.D
- new net GND: U$1.GND
- new net N$12: IC1.PC1, U$1.SCL
- new net N$13: IC1.PC0, U$1.SDA
- net +3.3V: now also U$1.VCC
- net +3.3V-IN: now also GND25.D
- net +5V-IN: now also GND28.D
Changed lines of the file:
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@@
 <part name="GND" library="medipix" deviceset="PIN" device="" value="GND"/>
 <part name="GND1" library="medipix" deviceset="PIN" device="" value="GND"/>
-<part name="TXD0" library="medipix" deviceset="PIN" device="" value="TX"/>
-<part name="RXD0" library="medipix" deviceset="PIN" device="" value="RX"/>
 <part name="+3.3V1" library="medipix" deviceset="+3.3V" device=""/>
 <part name="GND3" library="medipix" deviceset="GND" device=""/>
@@
 <part name="R34" library="medipix" deviceset="RESISTOR" device="0805" value="1k"/>
 <part name="R35" library="medipix" deviceset="RESISTOR" device="0805" value="1k"/>
-<part name="P3" library="con-molex-picoblade" deviceset="53398-0510" device=""/>
-<part name="P1" library="con-molex-picoblade" deviceset="53398-0310" device=""/>
-<part name="P2" library="con-molex-picoblade" deviceset="53398-0310" device=""/>
+<part name="P3" library="con-molex-picoblade" deviceset="53398-0510" device="" value="PICOBLADE"/>
+<part name="P1" library="con-molex-picoblade" deviceset="53398-0310" device="" value="PICOBLADE"/>
+<part name="P2" library="con-molex-picoblade" deviceset="53398-0310" device="" value="PICOBLADE"/>
 <part name="U18" library="medipix" deviceset="IRF7319" device=""/>
 <part name="R36" library="medipix" deviceset="RESISTOR" device="0805" value="100k"/>
@@
 <part name="TXD1" library="medipix" deviceset="PIN" device="" value="IN"/>
 <part name="TXD2" library="medipix" deviceset="PIN" device="" value="OUT"/>
+<part name="U$1" library="medipix" deviceset="THERM" device=""/>
+<part name="GND2" library="medipix" deviceset="GND" device=""/>
+<part name="+3.3V8" library="medipix" deviceset="+3.3V" device=""/>
+<part name="GND28" library="medipix" deviceset="PIN" device="" value="+5"/>
+<part name="GND25" library="medipix" deviceset="PIN" device="" value="+3.3"/>
 </parts>
 <sheets>
@@
 <instance part="GND" gate="A" x="12.7" y="151.13" rot="R180"/>
 <instance part="GND1" gate="A" x="12.7" y="147.32" rot="R180"/>
-<instance part="TXD0" gate="A" x="111.76" y="106.68"/>
-<instance part="RXD0" gate="A" x="111.76" y="114.3"/>
 <instance part="+3.3V1" gate="G$1" x="2.54" y="124.46"/>
 <instance part="GND3" gate="1" x="25.4" y="132.08"/>
@@
 <instance part="TXD1" gate="A" x="130.81" y="-48.26" rot="R270"/>
 <instance part="TXD2" gate="A" x="175.26" y="-27.94" rot="R90"/>
+<instance part="U$1" gate="G$1" x="139.7" y="139.7"/>
+<instance part="GND2" gate="1" x="127" y="129.54"/>
+<instance part="+3.3V8" gate="G$1" x="127" y="149.86"/>
+<instance part="GND28" gate="A" x="12.7" y="90.932"/>
+<instance part="GND25" gate="A" x="12.7" y="80.772"/>
 </instances>
 <busses>
@@
 <junction x="-88.9" y="63.5"/>
 </segment>
+<segment>
+<wire x1="7.62" y1="90.932" x2="7.62" y2="93.98" width="0.1524" layer="91"/>
+<pinref part="GND28" gate="A" pin="D"/>
+<label x="7.62" y="93.98" size="1.778" layer="95"/>
+</segment>
 </net>
 <net name="+3.3V-IN" class="0">
@@
 <pinref part="+3.3V4" gate="G$1" pin="+3.3V-IN"/>
 <junction x="-88.9" y="43.18"/>
+</segment>
+<segment>
+<pinref part="GND25" gate="A" pin="D"/>
+<wire x1="7.62" y1="83.82" x2="7.62" y2="80.772" width="0.1524" layer="91"/>
+<label x="7.62" y="83.82" size="1.778" layer="95"/>
 </segment>
 </net>
@@
 <junction x="220.98" y="88.9"/>
 </segment>
+<segment>
+<pinref part="U$1" gate="G$1" pin="VCC"/>
+<wire x1="129.54" y1="142.24" x2="127" y2="142.24" width="0.1524" layer="91"/>
+<wire x1="127" y1="142.24" x2="127" y2="147.32" width="0.1524" layer="91"/>
+<pinref part="+3.3V8" gate="G$1" pin="+3.3V"/>
+</segment>
 </net>
 <net name="N$8" class="0">
@@
 </segment>
 </net>
-<net name="N$10" class="0">
-<segment>
-<pinref part="IC1" gate="G$1" pin="PD3"/>
-<wire x1="93.98" y1="109.22" x2="101.6" y2="109.22" width="0.1524" layer="91"/>
-<wire x1="101.6" y1="109.22" x2="101.6" y2="106.68" width="0.1524" layer="91"/>
-<pinref part="TXD0" gate="A" pin="D"/>
-<wire x1="101.6" y1="106.68" x2="106.68" y2="106.68" width="0.1524" layer="91"/>
-</segment>
-</net>
-<net name="N$11" class="0">
-<segment>
-<pinref part="IC1" gate="G$1" pin="PD2"/>
-<pinref part="RXD0" gate="A" pin="D"/>
-<wire x1="93.98" y1="111.76" x2="106.68" y2="111.76" width="0.1524" layer="91"/>
-<wire x1="106.68" y1="111.76" x2="106.68" y2="114.3" width="0.1524" layer="91"/>
-</segment>
-</net>
 <net name="PA0" class="0">
 <segment>
@@
 </segment>
 </net>
+<net name="N$12" class="0">
+<segment>
+<pinref part="IC1" gate="G$1" pin="PC1"/>
+<pinref part="U$1" gate="G$1" pin="SCL"/>
+<wire x1="93.98" y1="137.16" x2="129.54" y2="137.16" width="0.1524" layer="91"/>
+</segment>
+</net>
+<net name="N$13" class="0">
+<segment>
+<pinref part="IC1" gate="G$1" pin="PC0"/>
+<pinref part="U$1" gate="G$1" pin="SDA"/>
+<wire x1="93.98" y1="139.7" x2="129.54" y2="139.7" width="0.1524" layer="91"/>
+</segment>
+</net>
+<net name="GND" class="0">
+<segment>
+<pinref part="U$1" gate="G$1" pin="GND"/>
+<wire x1="129.54" y1="134.62" x2="127" y2="134.62" width="0.1524" layer="91"/>
+<wire x1="127" y1="134.62" x2="127" y2="132.08" width="0.1524" layer="91"/>
+<pinref part="GND2" gate="1" pin="GND"/>
+</segment>
+</net>
